File: electronics/clock.sch (KiCad schematic (older format))
At the start: 6 parts, among them U7 LM555N

Commit message: Removed excess LEDs, updated library cache
Four LEDs should be enough for the incoming signals. This has the
advantage of using a 4015 less.
Parts:
- removed C5: 10u, ~, symbol CAPAPOL
- added C4: 10u, symbol CP
- renumbered C4 to C3, R28 to R16, R29 to R17, U7 to U5
Connections:
- net labels added: Clock
- net labels removed: Clk
- wire segments 26 -> 22
Changed lines of the file:
@@
 LIBS:valves
 LIBS:Gajda_cmosieee
-LIBS:LogicBoxen-cache
 EELAYER 25 0
 EELAYER END
@@
 $EndDescr
 $Comp
-L LM555N U7
+L LM555N U5
 U 1 1 555C383B
 P 4950 4450
-F 0 "U7" H 4950 4550 70  0000 C CNN
+F 0 "U5" H 4950 4550 70  0000 C CNN
 F 1 "LM555N" H 4950 4350 70  0000 C CNN
 F 2 "" H 4950 4450 60  0000 C CNN
@@
 $EndComp
 $Comp
-L C C4
+L C C3
 U 1 1 555C3847
 P 3700 4300
-F 0 "C4" H 3700 4400 40  0000 L CNN
+F 0 "C3" H 3700 4400 40  0000 L CNN
 F 1 "0.01u" H 3706 4215 40  0000 L CNN
 F 2 "~" H 3738 4150 30  0000 C CNN
@@
 $EndComp
 $Comp
-L R R29
+L R R17
 U 1 1 555C3853
 P 6300 4750
-F 0 "R29" V 6380 4750 40  0000 C CNN
+F 0 "R17" V 6380 4750 40  0000 C CNN
 F 1 "68k" V 6307 4751 40  0000 C CNN
 F 2 "~" V 6230 4750 30  0000 C CNN
 F 3 "~" H 6300 4750 30  0000 C CNN
 	1    6300 4750
-	1    0    0    -1
-$EndComp
-$Comp
-L CAPAPOL C5
-U 1 1 555C385F
-P 6300 5300
-F 0 "C5" H 6350 5400 40  0000 L CNN
-F 1 "10u" H 6350 5200 40  0000 L CNN
-F 2 "~" H 6400 5150 30  0000 C CNN
-F 3 "~" H 6300 5300 300 0000 C CNN
-	1    6300 5300
 	1    0    0    -1
 $EndComp
@@
 L GND #PWR016
 U 1 1 555C386B
-P 6300 5550
-F 0 "#PWR016" H 6300 5550 30  0001 C CNN
-F 1 "GND" H 6300 5480 30  0001 C CNN
-F 2 "" H 6300 5550 60  0000 C CNN
-F 3 "" H 6300 5550 60  0000 C CNN
-	1    6300 5550
+P 6300 5450
+F 0 "#PWR016" H 6300 5450 30  0001 C CNN
+F 1 "GND" H 6300 5380 30  0001 C CNN
+F 2 "" H 6300 5450 60  0000 C CNN
+F 3 "" H 6300 5450 60  0000 C CNN
+	1    6300 5450
 	1    0    0    -1
 $EndComp
 Text HLabel 6350 3500 2    60   Output ~ 0
-Clk
+Clock
 $Comp
-L R R28
+L R R16
 U 1 1 555CE354
 P 6200 3200
-F 0 "R28" V 6280 3200 40  0000 C CNN
+F 0 "R16" V 6280 3200 40  0000 C CNN
 F 1 "10k" V 6207 3201 40  0000 C CNN
 F 2 "~" V 6130 3200 30  0000 C CNN
@@
 $EndComp
 $Comp
-L VCC #PWR020
+L VCC #PWR017
 U 1 1 555CE368
 P 6200 2900
-F 0 "#PWR020" H 6200 3000 30  0001 C CNN
+F 0 "#PWR017" H 6200 3000 30  0001 C CNN
 F 1 "VCC" H 6200 3000 30  0000 C CNN
 F 2 "" H 6200 2900 60  0000 C CNN
@@
 	5650 4650 5900 4650
 Wire Wire Line
-	5900 3900 5900 4650
-Wire Wire Line
-	5900 4650 5900 5000
+	5900 3900 5900 5000
 Wire Wire Line
 	5900 3900 4150 3900
@@
 	4000 4500 4250 4500
 Wire Wire Line
-	3700 4500 3700 4550
+	3700 4450 3700 4550
 Wire Wire Line
-	6300 5000 6300 5100
+	6300 4900 6300 5100
 Wire Wire Line
-	6300 4400 6300 4450
+	6300 4400 6300 4600
 Wire Wire Line
-	6300 4450 6300 4500
-Wire Wire Line
-	6300 5500 6300 5550
+	6300 5400 6300 5450
 Wire Wire Line
 	6150 4150 6100 4100
@@
 	5650 3500 5650 4250
 Wire Wire Line
-	6250 3500 6250 3500
+	5650 3500 6350 3500
 Wire Wire Line
-	6250 3500 6200 3500
+	6200 2900 6200 3050
 Wire Wire Line
-	6200 3500 5650 3500
-Wire Wire Line
-	6350 3500 6250 3500
-Wire Wire Line
-	6200 2900 6200 2950
-Wire Wire Line
-	6200 3450 6200 3500
+	6200 3350 6200 3500
 Connection ~ 6200 3500
 Connection ~ 6300 4450
 NoConn ~ 6300 3900
+Wire Wire Line
+	3700 4100 3700 4150
+Connection ~ 6300 5000
+$Comp
+L CP C4
+U 1 1 5598FF7F
+P 6300 5250
+F 0 "C4" H 6325 5350 50  0000 L CNN
+F 1 "10u" H 6325 5150 50  0000 L CNN
+F 2 "" H 6338 5100 30  0000 C CNN
+F 3 "" H 6300 5250 60  0000 C CNN
+	1    6300 5250
+	1    0    0    -1
+$EndComp
 $EndSCHEMATC
